File: fenyjelző/SzineszFeny_V11.brd (EAGLE design)
At the start: 137.1 x 39 mm, 203 parts, among them CN3 PIN05_2'THT', IC1 BEM_VEDO, IC2 BEM_VEDO, IC3 BEM_VEDO, IC4 BEM_VEDO, IC5 BEM_VEDO, IC6 BEM_VEDO, IC7 SCT2168SOP16, IC8 SCT2168SOP16, IC9 SCT2168SOP16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

Commit message: fenyjelzo 90%os lett
Parts:
- moved C1 8.95 mm to (66.7, 34.1), flipped to the bottom
- moved C2 8.60 mm to (67.7, 28.8), flipped to the bottom
- moved Q2 5.08 mm to (67.8, 31.4), flipped to the bottom, turned to 0 degrees
- moved C3 4.13 mm to (71.9, 34.3), flipped to the bottom
- moved R109 2.54 mm to (65.0, 1.96)
- moved R112 2.54 mm to (65.0, 3.96)
- moved R113 2.54 mm to (65.0, 5.96)
- moved R116 2.54 mm to (65.0, 7.96)
- moved R107 2.54 mm to (65.0, 9.96)
- moved R108 2.54 mm to (65.0, 12.0)
- moved R106 2.27 mm to (63.5, 10.8)
- moved R105 2.27 mm to (65.5, 10.8)
- moved R114 2.27 mm to (67.5, 10.8)
- moved R115 2.27 mm to (69.5, 10.8)
- moved U1 1.59 mm to (74.2, 29.8)
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Connections:
- net GND renamed N$1
Routing:
- net RA5: track 0.00 -> 47.8 mm, vias 0 -> 1
- net RA0: track 10.2 -> 57.7 mm, vias 0 -> 3
- net RA1: track 6.75 -> 52.2 mm, vias 0 -> 3
- net RA3: track 4.78 -> 49.4 mm, vias 0 -> 3
- net RA2: track 2.56 -> 41.2 mm, vias 0 -> 3
- net N$1: track 624.6 -> 660.8 mm
- net RB5: track 10.8 -> 44.3 mm, vias 0 -> 3
- net RE2: track 19.3 -> 40.6 mm
- net RE1: track 21.8 -> 41.9 mm
- net RC5: track 54.0 -> 71.7 mm, vias 1 -> 2
- net RC2: track 194.2 -> 210.3 mm, vias 7 -> 8
- net RB4: track 14.3 -> 29.7 mm, vias 0 -> 2
- net RC3: track 204.2 -> 217.4 mm, vias 5 -> 6
- net RB2: track 0.00 -> 12.0 mm, vias 0 -> 1
- net +5V: track 564.1 -> 556.1 mm, vias 39 -> 41
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