File: fenyjelző/SzineszFeny_V11.sch (EAGLE design)
At the start: 203 parts, among them CN3 PIN05_2'THT', IC1 BEM_VEDO, IC2 BEM_VEDO, IC3 BEM_VEDO, IC4 BEM_VEDO, IC5 BEM_VEDO, IC6 BEM_VEDO, IC7 SCT2168SOP16, IC8 SCT2168SOP16, IC9 SCT2168SOP16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

Commit message: fenyjelzo 90%os lett
Connections:
- net GND renamed N$1
Changed lines of the file:
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@@
 </busses>
 <nets>
-<net name="GND" class="0">
+<net name="N$1" class="0">
 <segment>
 <pinref part="GND1" gate="1" pin="GND"/>
