File: MTX12Br/Mtx12BR_v1.1.sch (EAGLE design)
At the start: 118 parts, among them CN1 TESTCSAVAR3.5, CN2 PIN07_2, IC1 SCT2168SOP16, IC2 SCT2168SOP16, IC3 SCT2168SOP16, IC4 SCT2168SOP16, IC5 SCT2168SOP16, IC6 SCT2168SOP16, IC7 SCT2168SOP16, IC8 SCT2168SOP16, Q1 20MHz, Q2 BC846BSMD, SW1 SPG2, SW10 SPG2, SW11 SPG2, SW12 SPG2, SW2 SPG2, SW3 SPG2, SW4 SPG2, SW5 SPG2, SW6 SPG2, SW7 SPG2, SW8 SPG2, SW9 SPG2

Commit message: mtx12 30% kesz
Parts:
- removed IC1, IC2, IC3, IC4, IC5, IC6, IC7, IC8: SCT2168SOP16, Cf_IC:SCT2168SOP16
- added U$1, U$2, U$3, U$4, U$5, U$6, U$7, U$8: SCT2167SSOP, SCT2167:SCT2167SSOP
Connections:
- removed net N$109: DPL12.C, IC8.09_OUT4
- new net N$96: DL38.C, U$8.09_OUT4
- net +3V3: now also U$1.16_VDD, U$2.16_VDD, U$3.16_VDD, U$4.16_VDD, U$5.16_VDD, U$6.16_VDD, U$7.16_VDD, U$8.16_VDD; no longer IC1.16_VDD, IC2.16_VDD, IC3.16_VDD, IC4.16_VDD, IC5.16_VDD, IC6.16_VDD, IC7.16_VDD, IC8.16_VDD
- net GND: now also U$1.01_GND, U$2.01_GND, U$3.01_GND, U$4.01_GND, U$5.01_GND, U$6.01_GND, U$7.01_GND, U$8.01_GND; no longer IC1.01_GND, IC2.01_GND, IC3.01_GND, IC4.01_GND, IC5.01_GND, IC6.01_GND, IC7.01_GND, IC8.01_GND
- net N$10: now also U$4.10_OUT5; no longer IC5.10_OUT5
- net N$102: now also U$3.07_OUT2; no longer IC8.07_OUT2
- net N$103: now also U$3.06_OUT1; no longer IC8.06_OUT1
- net N$104: now also U$3.10_OUT5; no longer IC8.10_OUT5
- net N$105: now also U$3.11_OUT6; no longer IC8.11_OUT6
- net N$106: now also U$3.12_OUT7; no longer IC8.12_OUT7
- net N$107: now also U$3.08_OUT3; no longer IC8.08_OUT3
- net N$108: now also U$3.05_OUT0; no longer IC8.05_OUT0
- net N$11: now also U$4.06_OUT1; no longer IC5.06_OUT1
- net N$112: now also U$3.15_REXT; no longer IC8.15_REXT
- net N$115: now also U$1.14_SDO; no longer IC4.14_SDO
- net N$12: now also U$4.11_OUT6; no longer IC5.11_OUT6
- net N$13: now also U$6.06_OUT1; no longer IC7.06_OUT1
- net N$14: now also U$4.12_OUT7; no longer IC5.12_OUT7
- net N$15: now also U$6.10_OUT5; no longer IC7.10_OUT5
- net N$158: now also U$4.14_SDO, U$5.02_SDI; no longer IC5.14_SDO, IC6.02_SDI
- net N$16: now also U$6.11_OUT6; no longer IC7.11_OUT6
- net N$17: now also U$4.05_OUT0; no longer IC5.05_OUT0
- net N$19: now also U$4.09_OUT4; no longer IC5.09_OUT4
- net N$21: now also U$7.15_REXT; no longer IC2.15_REXT
- net N$22: now also U$6.12_OUT7; no longer IC7.12_OUT7
- net N$24: now also U$2.09_OUT4; no longer IC3.09_OUT4
- net N$26: now also U$6.08_OUT3; no longer IC7.08_OUT3
- net N$27: now also U$1.07_OUT2; no longer IC4.07_OUT2
- net N$28: now also U$1.06_OUT1; no longer IC4.06_OUT1
- net N$29: now also U$2.07_OUT2; no longer IC3.07_OUT2
- net N$30: now also U$2.06_OUT1; no longer IC3.06_OUT1
- net N$31: now also U$2.10_OUT5; no longer IC3.10_OUT5
- net N$32: now also U$2.11_OUT6; no longer IC3.11_OUT6
- net N$369: now also U$1.13_!OE!, U$2.13_!OE!, U$3.13_!OE!, U$4.13_!OE!, U$5.13_!OE!, U$6.13_!OE!, U$7.13_!OE!, U$8.13_!OE!; no longer IC1.13_!OE!, IC2.13_!OE!, IC3.13_!OE!, IC4.13_!OE!, IC5.13_!OE!, IC6.13_!OE!, IC7.13_!OE!, IC8.13_!OE!
- net N$37: now also U$8.15_REXT; no longer IC1.15_REXT
- net N$38: now also DPL8.C, U$5.09_OUT4; no longer DL36.C, IC1.07_OUT2
- net N$39: now also DPL10.C, U$6.09_OUT4; no longer DL37.C, IC1.08_OUT3
- net N$4: now also U$4.08_OUT3; no longer IC5.08_OUT3
- net N$40: now also DL11.C, U$7.05_OUT0; no longer DL38.C, IC1.09_OUT4
- net N$43: now also U$2.12_OUT7; no longer IC3.12_OUT7
- net N$46: now also DL12.C, U$7.06_OUT1; no longer DL39.C, IC1.10_OUT5
- net N$47: now also U$6.05_OUT0; no longer IC7.05_OUT0
- net N$48: now also DL13.C, U$7.07_OUT2; no longer DPL10.C, IC7.09_OUT4
- net N$49: now also U$5.14_SDO, U$6.02_SDI; no longer IC6.14_SDO, IC7.02_SDI
- net N$5: now also U$6.07_OUT2; no longer IC7.07_OUT2
- net N$50: now also U$2.08_OUT3; no longer IC3.08_OUT3
- net N$52: now also U$7.11_OUT6; no longer IC2.11_OUT6
- net N$53: now also U$7.02_SDI; no longer IC2.02_SDI
- net N$54: now also U$7.14_SDO, U$8.02_SDI; no longer IC1.02_SDI, IC2.14_SDO
- net N$55: now also U$7.12_OUT7; no longer IC2.12_OUT7
- net N$57: now also U$2.02_SDI, U$6.14_SDO; no longer IC3.02_SDI, IC7.14_SDO
- net N$58: now also U$2.05_OUT0; no longer IC3.05_OUT0
- net N$59: now also U$1.10_OUT5; no longer IC4.10_OUT5
- net N$6: now also DPL4.C, U$1.09_OUT4; no longer DL34.C, IC1.05_OUT0
- net N$60: now also U$6.15_REXT; no longer IC7.15_REXT
- net N$61: now also DL14.C, U$7.08_OUT3; no longer DL11.C, IC2.05_OUT0
- net N$63: now also U$2.14_SDO, U$3.02_SDI; no longer IC3.14_SDO, IC8.02_SDI
- net N$64: now also U$1.11_OUT6; no longer IC4.11_OUT6
- net N$65: now also U$1.12_OUT7; no longer IC4.12_OUT7
- net N$66: now also U$1.08_OUT3; no longer IC4.08_OUT3
- net N$67: now also U$1.05_OUT0; no longer IC4.05_OUT0
- net N$68: now also U$8.12_OUT7; no longer IC1.12_OUT7
- net N$69: now also U$8.11_OUT6; no longer IC1.11_OUT6
- net N$7: now also U$4.07_OUT2; no longer IC5.07_OUT2
- net N$70: now also U$5.07_OUT2; no longer IC6.07_OUT2
- net N$73: now also DL16.C, U$7.09_OUT4; no longer DL12.C, IC2.06_OUT1
- net N$74: now also U$5.06_OUT1; no longer IC6.06_OUT1
- net N$75: now also U$5.10_OUT5; no longer IC6.10_OUT5
- net N$76: now also U$5.11_OUT6; no longer IC6.11_OUT6
- net N$77: now also U$5.12_OUT7; no longer IC6.12_OUT7
- net N$78: now also U$5.08_OUT3; no longer IC6.08_OUT3
- net N$79: now also U$5.05_OUT0; no longer IC6.05_OUT0
- net N$8: now also DPL12.C, U$3.09_OUT4; no longer DL35.C, IC1.06_OUT1
- net N$81: now also U$1.02_SDI, U$3.14_SDO; no longer IC4.02_SDI, IC8.14_SDO
- net N$82: now also DL17.C, U$7.10_OUT5; no longer DPL4.C, IC4.09_OUT4
- net N$85: now also U$2.15_REXT; no longer IC3.15_REXT
- net N$86: now also DL34.C, U$8.05_OUT0; no longer DL13.C, IC2.07_OUT2
- net N$87: now also U$1.15_REXT; no longer IC4.15_REXT
- net N$88: now also U$4.15_REXT; no longer IC5.15_REXT
- net N$89: now also U$5.15_REXT; no longer IC6.15_REXT
- net N$90: now also DL35.C, U$8.06_OUT1; no longer DL14.C, IC2.08_OUT3
- net N$91: now also DL36.C, U$8.07_OUT2; no longer DL16.C, IC2.09_OUT4
- net N$92: now also DL37.C, U$8.08_OUT3; no longer DL17.C, IC2.10_OUT5
- net N$99: now also DL39.C, U$8.10_OUT5; no longer DPL8.C, IC6.09_OUT4
- net SCK3: now also U$1.03_CLK, U$2.03_CLK, U$3.03_CLK, U$4.03_CLK, U$5.03_CLK, U$6.03_CLK, U$7.03_CLK, U$8.03_CLK; no longer IC1.03_CLK, IC2.03_CLK, IC3.03_CLK, IC4.03_CLK, IC5.03_CLK, IC6.03_CLK, IC7.03_CLK, IC8.03_CLK
- net SDO2: now also U$4.02_SDI, U$8.14_SDO; no longer IC1.14_SDO, IC5.02_SDI
- net SS3: now also U$1.04_!LA!, U$2.04_!LA!, U$3.04_!LA!, U$4.04_!LA!, U$5.04_!LA!, U$6.04_!LA!, U$7.04_!LA!, U$8.04_!LA!; no longer IC1.04_!LA!, IC2.04_!LA!, IC3.04_!LA!, IC4.04_!LA!, IC5.04_!LA!, IC6.04_!LA!, IC7.04_!LA!, IC8.04_!LA!
