File: Streamnet_doboz/stream_i-o_2_3.brd (EAGLE design)
At the start: 192 x 74.5 mm, 225 parts, among them IC1 SCT21SOP16, IC12 LD117AS33TR, IC3 BEM_VEDO, IC4 7805TV, J1 PIN1-2, Q1 20MHz, T1 BD242, T10 BD242, T11 BD242, T12 BD242, T13 BD242, T14 BD242, T15 BD242, T16 BD242, T17 BC858, T2 BD242, T3 BD242, T4 BD242, T5 BD242, T6 BD242, T7 BD242, T8 BD242, T9 BD242, U1 MAX232SOIC16, U2 PIC32MX250F128B-I_SS

Commit message: stream_haladás
Parts:
- removed U$2, U$3, U$4: SCT21SOP16, StarChips:SOP16
- added U$1, U$10, U$7, U$8, U$9: SCT2167SSOP, SCT2167:SSOP
- moved R16 288.9 mm to (-168.9, 33.8), flipped to the bottom
- moved D20 288.6 mm to (-168.8, 37.5), flipped to the bottom
- moved LED16 287.7 mm to (-168.3, 35.7), flipped to the bottom
- moved ZOLD_2P8 281.2 mm to (-165.0, 10.7), flipped to the bottom
- moved ZOLD_4P16 281.2 mm to (-165.0, 24.5), flipped to the bottom
- moved T16 273.7 mm to (-161.3, 27.3), flipped to the top
- moved D19 262.9 mm to (-155.9, 36.8), flipped to the bottom
- moved R46 259.1 mm to (-154.0, 2.22), flipped to the top
- moved R47 259.1 mm to (-154.0, 4.76), flipped to the top
- moved ZOLD_2P7 257.2 mm to (-153.0, 10.7), flipped to the bottom
- moved ZOLD_4P15 257.2 mm to (-153.0, 24.5), flipped to the bottom
- moved LED15 256.5 mm to (-152.7, 34.0), flipped to the bottom
- moved T15 253.4 mm to (-151.1, 38.7), flipped to the top
- moved D31 250.8 mm to (-149.9, 17.1), flipped to the top
- moved D32 250.8 mm to (-149.9, 14.8), flipped to the top
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Connections:
- removed net N$102: OK4.13, U$3.6
- removed net N$136: U$3.14, U$4.2
- new net 01_GND: U$10.1, U$7.1, U$8.1, U$9.1
- new net 16_VDD: U$10.16, U$7.16, U$8.16, U$9.16
- new net N$97: OK4.13, U$7.6
- net +3V3: now also U$1.16; no longer U$2.16, U$3.16, U$4.16
- net CHECK: no longer U$4.14
- net CLK: now also U$1.3; no longer U$2.3, U$3.3, U$4.3
- net GND: now also U$1.1, U$1.13; no longer U$2.1, U$2.13, U$3.1, U$3.13, U$4.1, U$4.13
- net LABE: now also U$1.4; no longer U$2.4, U$3.4, U$4.4
- net N$100: now also U$8.11; no longer U$4.11
- net N$101: now also U$7.5; no longer U$3.5
- net N$103: now also U$7.7; no longer U$3.7
- net N$104: now also U$7.8; no longer U$3.8
- net N$113: now also U$8.12; no longer U$4.12
- net N$127: now also U$8.5; no longer U$4.5
- net N$128: now also U$8.6; no longer U$4.6
- net N$129: now also U$8.7; no longer U$4.7
- net N$130: now also U$8.8; no longer U$4.8
- net N$131: no longer U$4.15
- net N$132: no longer U$3.15
- net N$133: now also U$1.15; no longer U$2.15
- net N$134: now also U$1.2; no longer U$2.2
- net N$135: now also U$1.14; no longer U$2.14, U$3.2
- net N$64: now also U$1.9; no longer U$2.9
- net N$65: now also U$1.10; no longer U$2.10
- net N$66: now also U$1.11; no longer U$2.11
- net N$67: now also U$1.12; no longer U$2.12
- net N$76: now also U$8.9; no longer U$4.9
- net N$77: now also U$1.5; no longer U$2.5
- net N$78: now also U$1.6; no longer U$2.6
- net N$79: now also U$1.7; no longer U$2.7
- net N$80: now also U$1.8; no longer U$2.8
- net N$88: now also U$7.9; no longer U$3.9
- net N$89: now also U$7.10; no longer U$3.10
- net N$90: now also U$7.11; no longer U$3.11
- net N$91: now also U$7.12; no longer U$3.12
- net N$96: now also U$8.10; no longer U$4.10
Routing:
- net LABE: track 302.0 -> 142.3 mm, vias 5 -> 2
- net N$135: track 124.6 -> 0.00 mm, vias 2 -> 0
- net N$136: track 115.8 -> 0.00 mm, vias 2 -> 0
- net GND: track 909.1 -> 899.7 mm
- net +3V3: track 376.9 -> 367.8 mm
- net N$102: track 5.63 -> 0.00 mm
- net N$97: track 0.00 -> 5.04 mm
- net CLK: track 280.3 -> 276.1 mm
- net N$130: track 7.50 -> 3.89 mm
- net N$103: track 6.90 -> 3.61 mm
- net N$79: track 6.90 -> 3.77 mm
- net N$133: track 11.6 -> 9.51 mm
- net N$132: track 3.95 -> 2.08 mm
- net N$131: track 4.80 -> 3.30 mm
- net N$89: track 40.4 -> 39.0 mm
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- added copper zone on layer 1, net GND
- removed copper zone on layer 16, net GND
Other:
- board size 192 x 74.5 mm -> 287 x 74.5 mm

Commit message: streamnet ssopsodott
Parts:
- removed IC1, U$5: SCT21SOP16, StarChips:SOP16
- added D43, D44, D45, D46, D47, D48, D49, D50, D51, D52, D53, D54, D55, D56, D57, D58: (no value), dp_devices:SOD-123
- moved R16 272.4 mm to (103.5, 36.7), flipped to the top
- moved D20 272.1 mm to (103.3, 40.3), flipped to the top
- moved LED16 271.2 mm to (102.9, 38.6), flipped to the top
- moved U$8 267.2 mm to (70.3, 14.1), flipped to the bottom
- moved ZOLD_2P8 264.7 mm to (99.6, 13.6), flipped to the top
- moved ZOLD_4P16 264.7 mm to (99.6, 27.4), flipped to the top
- moved U$10 261.9 mm to (46.4, 32.4), flipped to the bottom, turned to 180 degrees
- moved U$7 260.0 mm to (70.5, 29.4), flipped to the bottom
- moved T16 257.2 mm to (95.9, 30.2), flipped to the bottom
- moved D19 246.4 mm to (90.5, 39.7), flipped to the top
- moved R46 242.6 mm to (88.6, 5.08), flipped to the bottom
- moved R47 242.6 mm to (88.6, 7.62), flipped to the bottom
- moved ZOLD_2P7 240.7 mm to (87.6, 13.6), flipped to the top
- moved ZOLD_4P15 240.7 mm to (87.6, 27.4), flipped to the top
- moved LED15 240.0 mm to (87.3, 36.8), flipped to the top
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Connections:
- removed net 01_GND: U$10.1, U$7.1, U$8.1, U$9.1
- removed net 16_VDD: U$10.16, U$7.16, U$8.16, U$9.16
- removed net GND: C10.2, C11.2, C12.2, C13.2, C14.2, C15.2, C16.2, C17.2, C4.2, C5.2, C6.1, C7.1, C8.-, C9.2, D41.A, D42.A, DC1.1, IC1.1, IC1.13, IC12.1, IC4.2, R17.1, R18.1, R43.1, R48.1, R49.1, R50.1, R51.1, R56.1, R67.2, SV1.1, U$1.1, U$1.13, U$5.1, U$5.13, U$6.6A, U$6.7A, U1.15, U2.19, U2.27, U2.8, ZOLD_2P1.1, ZOLD_2P2.1, ZOLD_2P3.1, ZOLD_2P4.1, ZOLD_2P5.1, ZOLD_2P6.1, ZOLD_2P7.1, ZOLD_2P8.1, ZOLD_3P1.1, ZOLD_3P2.1, ZOLD_4P1.1, ZOLD_4P1.3, ZOLD_4P10.1, ZOLD_4P10.3, ZOLD_4P11.1, ZOLD_4P11.3, ZOLD_4P12.1, ZOLD_4P12.3, ZOLD_4P13.1, ZOLD_4P13.3, ZOLD_4P14.1, ZOLD_4P14.3, ZOLD_4P15.1, ZOLD_4P15.3, ZOLD_4P16.1, ZOLD_4P16.3, ZOLD_4P17.1, ZOLD_4P2.1, ZOLD_4P2.3, ZOLD_4P3.1, ZOLD_4P3.3, ZOLD_4P4.1, ZOLD_4P4.3, ZOLD_4P5.1, ZOLD_4P5.3, ZOLD_4P6.1, ZOLD_4P6.3, ZOLD_4P7.1, ZOLD_4P7.3, ZOLD_4P8.1, ZOLD_4P8.3, ZOLD_4P9.1, ZOLD_4P9.3
- removed net N$131: R51.2
- removed net N$133: R49.2, U$1.15
- new net N$102: R50.1, U$7.15
- new net N$136: U$7.14, U$8.2
- new net N$156: R17.1, U$9.15
- new net N$171: R18.2, U$10.15
- net +3V3: now also U$10.16, U$7.16, U$8.16, U$9.16; no longer IC1.16, U$5.16
- net CHECK: now also U$8.13
- net CLK: now also U$10.3, U$7.3, U$8.3, U$9.3; no longer IC1.3, U$5.3
- net LABE: now also U$7.4, U$8.4
- net LAKI: now also U$10.4, U$9.4; no longer IC1.4, U$5.4
- net N$1: now also U$9.8; no longer IC1.8
- net N$10: now also D45.C
- net N$12: now also D46.C
- net N$13: now also U$9.9; no longer IC1.9
- net N$132: now also R51.1, U$8.15; no longer R50.2
- net N$134: now also U$10.14; no longer U$5.14
- net N$135: now also U$7.2
- net N$15: now also D47.C
- net N$16: now also U$9.10; no longer IC1.10
- net N$18: now also D48.C
- net N$19: now also U$9.11; no longer IC1.11
- net N$2: now also U$9.5; no longer IC1.5
- net N$21: now also D49.C
- net N$22: now also U$9.12; no longer IC1.12
- net N$24: now also D50.C
- net N$25: now also R49.1, U$1.15; no longer IC1.15, R17.2
- net N$26: now also C10.2, C11.2, C12.2, C13.2, C14.2, C15.2, C16.2, C17.2, C4.2, C5.2, C6.1, C7.1, C8.-, C9.2, D41.A, D42.A, D43.A, D44.A, D45.A, D46.A, D47.A, D48.A, D49.A, D50.A, D51.A, D52.A, D53.A, D54.A, D55.A, D56.A, D57.A, D58.A, DC1.1, IC12.1, IC4.2, R17.2, R18.1, R43.1, R48.1, R49.2, R50.2, R51.2, R56.1, R67.2, SV1.1, U$1.1, U$1.13, U$10.1, U$10.13, U$6.6A, U$6.7A, U$7.1, U$7.13, U$8.1, U$8.14, U$9.1, U$9.13, U1.15, U2.19, U2.27, U2.8, ZOLD_2P1.1, ZOLD_2P2.1, ZOLD_2P3.1, ZOLD_2P4.1, ZOLD_2P5.1, ZOLD_2P6.1, ZOLD_2P7.1, ZOLD_2P8.1, ZOLD_3P1.1, ZOLD_3P2.1, ZOLD_4P1.1, ZOLD_4P1.3, ZOLD_4P10.1, ZOLD_4P10.3, ZOLD_4P11.1, ZOLD_4P11.3, ZOLD_4P12.1, ZOLD_4P12.3, ZOLD_4P13.1, ZOLD_4P13.3, ZOLD_4P14.1, ZOLD_4P14.3, ZOLD_4P15.1, ZOLD_4P15.3, ZOLD_4P16.1, ZOLD_4P16.3, ZOLD_4P17.1, ZOLD_4P2.1, ZOLD_4P2.3, ZOLD_4P3.1, ZOLD_4P3.3, ZOLD_4P4.1, ZOLD_4P4.3, ZOLD_4P5.1, ZOLD_4P5.3, ZOLD_4P6.1, ZOLD_4P6.3, ZOLD_4P7.1, ZOLD_4P7.3, ZOLD_4P8.1, ZOLD_4P8.3, ZOLD_4P9.1, ZOLD_4P9.3; no longer R18.2, U$5.15
- net N$27: now also U$10.2, U$9.14; no longer IC1.14, U$5.2
- net N$33: now also U$10.5; no longer U$5.5
- net N$35: now also D51.C
- net N$36: now also U$10.6; no longer U$5.6
- net N$38: now also D52.C
- net N$39: now also U$10.7; no longer U$5.7
- net N$4: now also D43.C
- net N$41: now also D53.C
- net N$42: now also U$10.8; no longer U$5.8
- net N$44: now also D54.C
- net N$45: now also U$10.9; no longer U$5.9
- net N$47: now also D55.C
- net N$48: now also U$10.10; no longer U$5.10
- net N$5: now also U$9.6; no longer IC1.6
- net N$50: now also D56.C
- net N$51: now also U$10.11; no longer U$5.11
- net N$53: now also D57.C
- net N$54: now also U$10.12; no longer U$5.12
- net N$56: now also D58.C
- net N$7: now also D44.C
- net N$8: now also U$9.7; no longer IC1.7
- net SDO1: now also U$9.2; no longer IC1.2
Routing:
- net GND: track 899.7 -> 0.00 mm, vias 16 -> 0
- net N$26: track 4.77 -> 880.7 mm, vias 0 -> 18
- net LABE: track 142.3 -> 270.4 mm, vias 2 -> 5
- net N$135: track 0.00 -> 115.6 mm, vias 0 -> 2
- net N$136: track 0.00 -> 22.0 mm, vias 0 -> 2
- net +3V3: track 367.8 -> 387.7 mm, vias 9 -> 11
- net CLK: track 276.1 -> 288.9 mm
- net N$133: track 9.51 -> 0.00 mm
- net N$171: track 0.00 -> 7.49 mm
- net N$102: track 0.00 -> 7.07 mm, vias 0 -> 1
- net N$130: track 3.89 -> 9.35 mm
- net N$79: track 3.77 -> 8.43 mm
- net N$103: track 3.61 -> 7.72 mm
- net N$27: track 104.3 -> 108.0 mm
- net SDO1: track 39.6 -> 43.2 mm
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- added copper zone on layer 16, net N$26
- removed copper zone on layer 1, net GND
Other:
- board size 287 x 74.5 mm -> 202.4 x 71.6 mm

Commit message: stream testatkot megszunt
Parts:
- moved D43 199.7 mm to (114.1, 31.4), flipped to the top
- moved IC4 197.2 mm to (112.9, 15.2), flipped to the top
- moved D5 195.6 mm to (112.1, 40.3), flipped to the bottom
- moved LED1 195.6 mm to (112.1, 38.6), flipped to the bottom
- moved R1 195.6 mm to (112.1, 36.7), flipped to the bottom
- moved C8 193.7 mm to (111.1, 6.67), flipped to the top
- moved C9 189.9 mm to (109.2, 6.83), flipped to the bottom
- moved ZOLD_4P1 189.3 mm to (108.9, 27.4), flipped to the bottom
- moved T1 181.6 mm to (105.1, 30.2), flipped to the top
- moved R16 178.4 mm to (-74.9, 36.7), flipped to the bottom
- moved D20 178.1 mm to (-74.8, 40.3), flipped to the bottom
- moved DC1 177.3 mm to (102.9, 11.2), flipped to the bottom
- moved LED16 177.2 mm to (-74.3, 38.6), flipped to the bottom
- moved ZOLD_2P8 170.7 mm to (-71.1, 13.6), flipped to the bottom
- moved ZOLD_4P16 170.7 mm to (-71.1, 27.4), flipped to the bottom
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Routing:
- net U2RX: track 61.6 -> 74.3 mm
- net N$26: track 880.7 -> 890.6 mm
- net +5V: track 431.0 -> 438.3 mm
- net N$75: track 24.2 -> 18.1 mm
- added copper zone on layer 1, net N$26
- removed copper zone on layer 16, net N$26
Other:
- board size 202.4 x 71.6 mm -> 193.1 x 71.6 mm
- board text removed: "GND ATKOT"

Commit message: javult meg ez az
Parts:
- moved D43 1.59 mm to (112.6, 31.4)
- moved R1 0.22 mm to (112.2, 36.5), turned to 180 degrees
Routing:
- net N$26: track 890.6 -> 874.7 mm
- net +12V: track 524.4 -> 518.8 mm, vias 26 -> 24
- net N$4: track 7.09 -> 11.2 mm
- net N$3: track 18.3 -> 15.1 mm
Changed lines of the file:
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@@
 <attribute name="VALUE" x="97.4725" y="35.2425" size="1.27" layer="27" ratio="10" rot="R270"/>
 </element>
-<element name="R1" library="rcl" package="R0805" value="6R8" x="112.0775" y="36.67125" smashed="yes" rot="MR0">
-<attribute name="NAME" x="114.3" y="35.8775" size="0.8128" layer="26" font="vector" ratio="15" rot="MR90"/>
-<attribute name="VALUE" x="112.7125" y="34.13125" size="1.27" layer="28" rot="MR0"/>
+<element name="R1" library="rcl" package="R0805" value="6R8" x="112.23625" y="36.5125" smashed="yes" rot="MR180">
+<attribute name="NAME" x="110.01375" y="37.30625" size="0.8128" layer="26" font="vector" ratio="15" rot="MR270"/>
+<attribute name="VALUE" x="111.60125" y="39.0525" size="1.27" layer="28" rot="MR180"/>
 </element>
 <element name="LED1" library="led" package="CHIPLED_1206" value="RED" x="112.0775" y="38.57625" smashed="yes" rot="MR270">
@@
 <element name="U$9" library="SCT2167" package="SSOP" value="SCT2167SSOP" x="78.89875" y="34.13125" rot="R180"/>
 <element name="U$10" library="SCT2167" package="SSOP" value="SCT2167SSOP" x="-17.78" y="32.385" rot="R180"/>
-<element name="D43" library="dp_devices" package="SOD-123" value="" x="114.14125" y="31.4325" rot="R270"/>
+<element name="D43" library="dp_devices" package="SOD-123" value="" x="112.55375" y="31.4325" rot="R270"/>
 <element name="D44" library="dp_devices" package="SOD-123" value="" x="98.7425" y="31.4325" rot="R270"/>
 <element name="D45" library="dp_devices" package="SOD-123" value="" x="90.32875" y="31.59125" rot="MR270"/>
@@
 <contactref element="T1" pad="3"/>
 <contactref element="R1" pad="1"/>
-<wire x1="109.37875" y1="30.7975" x2="107.47375" y2="30.7975" width="0.3048" layer="16"/>
-<wire x1="107.47375" y1="30.7975" x2="106.83875" y2="30.1625" width="0.3048" layer="16"/>
+<wire x1="107.79125" y1="31.115" x2="106.83875" y2="30.1625" width="0.3048" layer="16"/>
 <wire x1="106.83875" y1="30.1625" x2="106.83875" y2="28.575" width="0.3048" layer="16"/>
 <wire x1="106.83875" y1="28.575" x2="105.88625" y2="27.6225" width="0.3048" layer="16"/>
 <wire x1="105.88625" y1="27.6225" x2="102.5525" y2="27.6225" width="0.3048" layer="16"/>
-<wire x1="109.37875" y1="30.7975" x2="110.01375" y2="30.1625" width="0.3048" layer="16"/>
-<wire x1="110.01375" y1="30.1625" x2="110.8075" y2="30.1625" width="0.3048" layer="16"/>
-<wire x1="110.8075" y1="30.1625" x2="111.4425" y2="30.7975" width="0.3048" layer="16"/>
-<wire x1="111.4425" y1="30.7975" x2="111.4425" y2="33.02" width="0.3048" layer="16"/>
-<wire x1="111.4425" y1="33.02" x2="112.55375" y2="34.13125" width="0.3048" layer="16"/>
-<wire x1="112.55375" y1="34.13125" x2="112.55375" y2="35.08375" width="0.3048" layer="16"/>
-<wire x1="112.55375" y1="35.08375" x2="113.18875" y2="35.71875" width="0.3048" layer="16"/>
-<wire x1="113.18875" y1="35.71875" x2="113.18875" y2="36.61" width="0.3048" layer="16"/>
-<wire x1="113.18875" y1="36.61" x2="113.1275" y2="36.67125" width="0.3048" layer="16"/>
+<wire x1="107.79125" y1="31.115" x2="108.9025" y2="31.115" width="0.3048" layer="16"/>
+<wire x1="108.9025" y1="31.115" x2="110.1725" y2="32.385" width="0.3048" layer="16"/>
+<wire x1="110.1725" y1="32.385" x2="110.1725" y2="34.6075" width="0.3048" layer="16"/>
+<wire x1="110.1725" y1="34.6075" x2="111.18625" y2="35.62125" width="0.3048" layer="16"/>
+<wire x1="111.18625" y1="35.62125" x2="111.18625" y2="36.5125" width="0.3048" layer="16"/>
 </signal>
 <signal name="N$4">
@@
 <wire x1="106.89125" y1="33.0725" x2="108.435" y2="33.0725" width="0.3048" layer="16"/>
 <contactref element="D43" pad="C"/>
-<wire x1="108.435" y1="33.0725" x2="114.14125" y2="33.0675" width="0" layer="19" extent="1-1"/>
+<wire x1="108.435" y1="33.0725" x2="108.44" y2="33.0675" width="0.6096" layer="1"/>
+<wire x1="108.44" y1="33.0675" x2="112.55375" y2="33.0675" width="0.6096" layer="1"/>
 </signal>
 <signal name="+12V">
@@
 <wire x1="88.9" y1="35.56" x2="89.2175" y2="35.8775" width="0.3048" layer="16"/>
 <wire x1="89.2175" y1="35.8775" x2="89.2175" y2="39.6875" width="0.3048" layer="16"/>
-<via x="105.56875" y="26.035" extent="1-16" drill="0.6096"/>
 <wire x1="-32.8" y1="36.83" x2="-32.8" y2="35.81625" width="0.3048" layer="16"/>
 <wire x1="-32.8" y1="35.81625" x2="-32.54375" y2="35.56" width="0.3048" layer="16"/>
@@
 <wire x1="84.455" y1="4.1275" x2="84.93125" y2="4.1275" width="0.6096" layer="16"/>
 <wire x1="84.93125" y1="4.1275" x2="85.24875" y2="4.28625" width="0.6096" layer="16"/>
-<wire x1="105.7275" y1="29.845" x2="105.7275" y2="26.19375" width="0.6096" layer="1"/>
-<wire x1="105.7275" y1="26.19375" x2="105.56875" y2="26.035" width="0.6096" layer="1"/>
-<wire x1="105.7275" y1="29.845" x2="107.15625" y2="31.27375" width="0.6096" layer="1"/>
-<wire x1="107.15625" y1="31.27375" x2="110.49" y2="31.27375" width="0.6096" layer="1"/>
-<via x="110.49" y="31.27375" extent="1-16" drill="0.6096"/>
 <wire x1="97.0575" y1="36.83" x2="97.0575" y2="35.6575" width="0.6096" layer="16"/>
 <via x="100.33" y="34.29" extent="1-16" drill="0.6096"/>
@@
 <wire x1="84.93125" y1="4.1275" x2="84.455" y2="4.1275" width="0.6096" layer="1"/>
 <wire x1="109.69625" y1="27.305" x2="106.83875" y2="27.305" width="0.9144" layer="16"/>
-<wire x1="106.83875" y1="27.305" x2="105.56875" y2="26.035" width="0.9144" layer="16"/>
-<wire x1="105.56875" y1="26.035" x2="104.93375" y2="25.4" width="0.9144" layer="16"/>
+<wire x1="106.83875" y1="27.305" x2="104.93375" y2="25.4" width="0.9144" layer="16"/>
 <wire x1="101.44125" y1="25.4" x2="100.48875" y2="26.3525" width="0.9144" layer="16"/>
 <wire x1="100.48875" y1="26.3525" x2="100.48875" y2="34.13125" width="0.9144" layer="16"/>
@@
 <wire x1="111.125" y1="20.0025" x2="111.125" y2="18.57375" width="1.016" layer="16"/>
 <wire x1="111.125" y1="18.57375" x2="110.33125" y2="17.78" width="1.016" layer="16"/>
-<wire x1="110.49" y1="31.27375" x2="110.49" y2="35.08375" width="0.8128" layer="16"/>
 <wire x1="-73.88" y1="36.67125" x2="-73.88" y2="37.24125" width="0.6096" layer="16"/>
 <wire x1="-73.88" y1="37.24125" x2="-72.545" y2="38.57625" width="0.6096" layer="16"/>
@@
 <via x="-70.485" y="34.925" extent="1-16" drill="0.6"/>
 <wire x1="-70.485" y1="34.925" x2="-69.69125" y2="34.925" width="0.8128" layer="1"/>
-<wire x1="110.49" y1="35.08375" x2="110.96625" y2="35.56" width="0.8128" layer="16"/>
-<wire x1="110.96625" y1="35.56" x2="110.96625" y2="36.61" width="0.8128" layer="16"/>
-<wire x1="110.96625" y1="36.61" x2="111.0275" y2="36.67125" width="0.8128" layer="16"/>
-<wire x1="113.8275" y1="38.57625" x2="112.7125" y2="38.57625" width="0.6096" layer="16"/>
-<wire x1="112.7125" y1="38.57625" x2="111.60125" y2="37.465" width="0.6096" layer="16"/>
-<wire x1="111.60125" y1="37.465" x2="111.60125" y2="37.245" width="0.6096" layer="16"/>
-<wire x1="111.60125" y1="37.245" x2="111.0275" y2="36.67125" width="0.6096" layer="16"/>
 <wire x1="28.09875" y1="33.81375" x2="29.27125" y2="33.81375" width="0.8128" layer="1"/>
 <wire x1="29.27125" y1="33.81375" x2="30.54125" y2="33.81375" width="0.8128" layer="16"/>
@@
 <wire x1="30.48" y1="33.7525" x2="29.3325" y2="33.7525" width="0.3048" layer="1"/>
 <wire x1="29.3325" y1="33.7525" x2="29.27125" y2="33.81375" width="0.3048" layer="1"/>
+<wire x1="109.69625" y1="27.305" x2="111.125" y2="28.73375" width="0.6096" layer="16"/>
+<wire x1="111.125" y1="28.73375" x2="111.125" y2="33.9725" width="0.6096" layer="16"/>
+<wire x1="111.125" y1="33.9725" x2="113.28625" y2="36.13375" width="0.6096" layer="16"/>
+<wire x1="113.28625" y1="36.13375" x2="113.28625" y2="36.5125" width="0.6096" layer="16"/>
+<wire x1="113.28625" y1="36.5125" x2="113.8275" y2="37.05375" width="0.6096" layer="16"/>
+<wire x1="113.8275" y1="37.05375" x2="113.8275" y2="38.57625" width="0.6096" layer="16"/>
 </signal>
 <signal name="N$5">
@@
 <contactref element="IC4" pad="2"/>
 <wire x1="96.14125" y1="7.14375" x2="96.14125" y2="5.23875" width="0.9144" layer="16"/>
-<wire x1="108.435" y1="29.2625" x2="112.13" y2="29.2625" width="0.6096" layer="1"/>
-<wire x1="112.13" y1="29.2625" x2="113.03" y2="30.1625" width="0.6096" layer="1"/>
-<wire x1="113.03" y1="30.1625" x2="113.03" y2="33.655" width="0.6096" layer="1"/>
-<wire x1="113.03" y1="33.655" x2="111.4425" y2="35.2425" width="0.6096" layer="1"/>
-<wire x1="111.4425" y1="35.2425" x2="105.7275" y2="35.2425" width="0.6096" layer="1"/>
-<wire x1="105.7275" y1="35.2425" x2="104.4575" y2="33.9725" width="0.6096" layer="1"/>
-<wire x1="104.4575" y1="33.9725" x2="104.4575" y2="26.9875" width="0.6096" layer="1"/>
-<wire x1="104.4575" y1="26.9875" x2="103.1875" y2="25.7175" width="0.6096" layer="1"/>
-<wire x1="103.1875" y1="25.7175" x2="99.98" y2="25.7175" width="0.6096" layer="1"/>
+<wire x1="104.89" y1="25.7175" x2="99.98" y2="25.7175" width="0.6096" layer="1"/>
 <wire x1="99.98" y1="25.7175" x2="96.435" y2="29.2625" width="0.6096" layer="1"/>
 <wire x1="96.99625" y1="11.43" x2="96.8375" y2="11.43" width="0.9144" layer="16"/>
@@
 <wire x1="62.07125" y1="15.875" x2="62.07125" y2="12.3825" width="1.6764" layer="1"/>
 <wire x1="60.435" y1="21.6425" x2="60.48375" y2="21.59375" width="1.6764" layer="1"/>
-<wire x1="113.03" y1="30.1625" x2="114.14125" y2="29.7975" width="0" layer="19" extent="1-1"/>
 <wire x1="53.6575" y1="29.7975" x2="53.49875" y2="30.48" width="0" layer="19" extent="1-16"/>
 <wire x1="78.105" y1="30.90875" x2="79.79" y2="30.48" width="0" layer="19" extent="1-16"/>
@@
 <wire x1="-50.4825" y1="67.51625" x2="-46.355" y2="67.51625" width="0" layer="19" extent="1-1"/>
 <wire x1="-54.61" y1="67.51625" x2="-50.4825" y2="67.51625" width="0" layer="19" extent="1-1"/>
+<wire x1="112.55375" y1="29.7975" x2="112.01875" y2="29.2625" width="0.6096" layer="1"/>
+<wire x1="112.01875" y1="29.2625" x2="108.435" y2="29.2625" width="0.6096" layer="1"/>
+<wire x1="104.89" y1="25.7175" x2="108.435" y2="29.2625" width="0.6096" layer="1"/>
 </signal>
 </signals>
