File: Streamnet_doboz/stream_i-o_2_3.sch (EAGLE design)
At the start: 225 parts, among them IC1 SCT21SOP16, IC12 LD117AS33TR, IC3 BEM_VEDO, IC4 7805TV, J1 PIN1-2, Q1 20MHz, T1 BD242, T10 BD242, T11 BD242, T12 BD242, T13 BD242, T14 BD242, T15 BD242, T16 BD242, T17 BC858, T2 BD242, T3 BD242, T4 BD242, T5 BD242, T6 BD242, T7 BD242, T8 BD242, T9 BD242, U1 MAX232SOIC16, U2 PIC32MX250F128B-I_SS

Commit message: stream_haladás
Parts:
- removed U$2, U$3, U$4: SCT21SOP16, StarChips:SCT21SOP16
- added U$1, U$10, U$7, U$8, U$9: SCT2167SSOP, SCT2167:SCT2167SSOP
Connections:
- removed net N$102: OK4B.EMIT, U$3.OUT1
- removed net N$136: U$3.SDO, U$4.SDI
- new net N$97: OK4B.EMIT, U$7.06_OUT1
- net +3V3: now also U$1.16_VDD; no longer U$2.VDD, U$3.VDD, U$4.VDD
- net CHECK: no longer U$4.SDO
- net CLK: now also U$1.03_CLK; no longer U$2.CLK, U$3.CLK, U$4.CLK
- net GND: now also U$1.01_GND, U$1.13_!OE!; no longer U$2.!OE, U$2.GND, U$3.!OE, U$3.GND, U$4.!OE, U$4.GND
- net LABE: now also U$1.04_!LA!; no longer U$2.!LA, U$3.!LA, U$4.!LA
- net N$100: now also U$8.11_OUT6; no longer U$4.OUT6
- net N$101: now also U$7.05_OUT0; no longer U$3.OUT0
- net N$103: now also U$7.07_OUT2; no longer U$3.OUT2
- net N$104: now also U$7.08_OUT3; no longer U$3.OUT3
- net N$113: now also U$8.12_OUT7; no longer U$4.OUT7
- net N$127: now also U$8.05_OUT0; no longer U$4.OUT0
- net N$128: now also U$8.06_OUT1; no longer U$4.OUT1
- net N$129: now also U$8.07_OUT2; no longer U$4.OUT2
- net N$130: now also U$8.08_OUT3; no longer U$4.OUT3
- net N$131: no longer U$4.REXT
- net N$132: no longer U$3.REXT
- net N$133: now also U$1.15_REXT; no longer U$2.REXT
- net N$134: now also U$1.02_SDI; no longer U$2.SDI
- net N$135: now also U$1.14_SDO; no longer U$2.SDO, U$3.SDI
- net N$64: now also U$1.09_OUT4; no longer U$2.OUT4
- net N$65: now also U$1.10_OUT5; no longer U$2.OUT5
- net N$66: now also U$1.11_OUT6; no longer U$2.OUT6
- net N$67: now also U$1.12_OUT7; no longer U$2.OUT7
- net N$76: now also U$8.09_OUT4; no longer U$4.OUT4
- net N$77: now also U$1.05_OUT0; no longer U$2.OUT0
- net N$78: now also U$1.06_OUT1; no longer U$2.OUT1
- net N$79: now also U$1.07_OUT2; no longer U$2.OUT2
- net N$80: now also U$1.08_OUT3; no longer U$2.OUT3
- net N$88: now also U$7.09_OUT4; no longer U$3.OUT4
- net N$89: now also U$7.10_OUT5; no longer U$3.OUT5
- net N$90: now also U$7.11_OUT6; no longer U$3.OUT6
- net N$91: now also U$7.12_OUT7; no longer U$3.OUT7
- net N$96: now also U$8.10_OUT5; no longer U$4.OUT5
Other:
- moved on the sheet: R49

Commit message: streamnet ssopsodott
Parts:
- removed IC1, U$5: SCT21SOP16, StarChips:SCT21SOP16
- added D43, D44, D45, D46, D47, D48, D49, D50, D51, D52, D53, D54, D55, D56, D57, D58: (no value), dp_devices:DIODE-SOD-123
Connections:
- removed net GND: C10.2, C11.2, C12.2, C13.2, C14.2, C15.2, C16.2, C17.2, C4.2, C5.2, C6.1, C7.1, C8.-, C9.2, D41.A, D42.A, DC1_GND.1, IC1.!OE, IC1.GND, IC12.ADJ, IC4.GND, R17.1, R18.1, R43.1, R48.1, R49.1, R50.1, R51.1, R56.1, R67.2, SV1.1, U$1.01_GND, U$1.13_!OE!, U$5.!OE, U$5.GND, U$6.11, U$6.13, U1.GND, U2.AVSS, U2.VSS, U2.VSS_2, ZOLD_2P1_1.1, ZOLD_2P2_1.1, ZOLD_2P3_1.1, ZOLD_2P4_1.1, ZOLD_2P5_1.1, ZOLD_2P6_1.1, ZOLD_2P7_1.1, ZOLD_2P8_1.1, ZOLD_3P1_1.1, ZOLD_3P2_1.1, ZOLD_4P10_1.1, ZOLD_4P10_3.1, ZOLD_4P11_1.1, ZOLD_4P11_3.1, ZOLD_4P12_1.1, ZOLD_4P12_3.1, ZOLD_4P13_1.1, ZOLD_4P13_3.1, ZOLD_4P14_1.1, ZOLD_4P14_3.1, ZOLD_4P15_1.1, ZOLD_4P15_3.1, ZOLD_4P16_1.1, ZOLD_4P16_3.1, ZOLD_4P17_1.1, ZOLD_4P1_1.1, ZOLD_4P1_3.1, ZOLD_4P2_1.1, ZOLD_4P2_3.1, ZOLD_4P3_1.1, ZOLD_4P3_3.1, ZOLD_4P4_1.1, ZOLD_4P4_3.1, ZOLD_4P5_1.1, ZOLD_4P5_3.1, ZOLD_4P6_1.1, ZOLD_4P6_3.1, ZOLD_4P7_1.1, ZOLD_4P7_3.1, ZOLD_4P8_1.1, ZOLD_4P8_3.1, ZOLD_4P9_1.1, ZOLD_4P9_3.1
- removed net N$131: R51.2
- removed net N$133: R49.2, U$1.15_REXT
- new net N$102: R50.1, U$7.15_REXT
- new net N$136: U$7.14_SDO, U$8.02_SDI
- new net N$156: R17.1, U$9.15_REXT
- new net N$171: R18.2, U$10.15_REXT
- net +3V3: now also U$10.16_VDD, U$7.16_VDD, U$8.16_VDD, U$9.16_VDD; no longer IC1.VDD, U$5.VDD
- net CHECK: now also U$8.13_!OE!
- net CLK: now also U$10.03_CLK, U$7.03_CLK, U$8.03_CLK, U$9.03_CLK; no longer IC1.CLK, U$5.CLK
- net LABE: now also U$7.04_!LA!, U$8.04_!LA!
- net LAKI: now also U$10.04_!LA!, U$9.04_!LA!; no longer IC1.!LA, U$5.!LA
- net N$1: now also U$9.08_OUT3; no longer IC1.OUT3
- net N$10: now also D45.C
- net N$12: now also D46.C
- net N$13: now also U$9.09_OUT4; no longer IC1.OUT4
- net N$132: now also R51.1, U$8.15_REXT; no longer R50.2
- net N$134: now also U$10.14_SDO; no longer U$5.SDO
- net N$135: now also U$7.02_SDI
- net N$15: now also D47.C
- net N$16: now also U$9.10_OUT5; no longer IC1.OUT5
- net N$18: now also D48.C
- net N$19: now also U$9.11_OUT6; no longer IC1.OUT6
- net N$2: now also U$9.05_OUT0; no longer IC1.OUT0
- net N$21: now also D49.C
- net N$22: now also U$9.12_OUT7; no longer IC1.OUT7
- net N$24: now also D50.C
- net N$25: now also R49.1, U$1.15_REXT; no longer IC1.REXT, R17.2
- net N$26: now also C10.2, C11.2, C12.2, C13.2, C14.2, C15.2, C16.2, C17.2, C4.2, C5.2, C6.1, C7.1, C8.-, C9.2, D41.A, D42.A, D43.A, D44.A, D45.A, D46.A, D47.A, D48.A, D49.A, D50.A, D51.A, D52.A, D53.A, D54.A, D55.A, D56.A, D57.A, D58.A, DC1_GND.1, IC12.ADJ, IC4.GND, R17.2, R18.1, R43.1, R48.1, R49.2, R50.2, R51.2, R56.1, R67.2, SV1.1, U$1.01_GND, U$1.13_!OE!, U$10.01_GND, U$10.13_!OE!, U$6.11, U$6.13, U$7.01_GND, U$7.13_!OE!, U$8.01_GND, U$8.14_SDO, U$9.01_GND, U$9.13_!OE!, U1.GND, U2.AVSS, U2.VSS, U2.VSS_2, ZOLD_2P1_1.1, ZOLD_2P2_1.1, ZOLD_2P3_1.1, ZOLD_2P4_1.1, ZOLD_2P5_1.1, ZOLD_2P6_1.1, ZOLD_2P7_1.1, ZOLD_2P8_1.1, ZOLD_3P1_1.1, ZOLD_3P2_1.1, ZOLD_4P10_1.1, ZOLD_4P10_3.1, ZOLD_4P11_1.1, ZOLD_4P11_3.1, ZOLD_4P12_1.1, ZOLD_4P12_3.1, ZOLD_4P13_1.1, ZOLD_4P13_3.1, ZOLD_4P14_1.1, ZOLD_4P14_3.1, ZOLD_4P15_1.1, ZOLD_4P15_3.1, ZOLD_4P16_1.1, ZOLD_4P16_3.1, ZOLD_4P17_1.1, ZOLD_4P1_1.1, ZOLD_4P1_3.1, ZOLD_4P2_1.1, ZOLD_4P2_3.1, ZOLD_4P3_1.1, ZOLD_4P3_3.1, ZOLD_4P4_1.1, ZOLD_4P4_3.1, ZOLD_4P5_1.1, ZOLD_4P5_3.1, ZOLD_4P6_1.1, ZOLD_4P6_3.1, ZOLD_4P7_1.1, ZOLD_4P7_3.1, ZOLD_4P8_1.1, ZOLD_4P8_3.1, ZOLD_4P9_1.1, ZOLD_4P9_3.1; no longer R18.2, U$5.REXT
- net N$27: now also U$10.02_SDI, U$9.14_SDO; no longer IC1.SDO, U$5.SDI
- net N$33: now also U$10.05_OUT0; no longer U$5.OUT0
- net N$35: now also D51.C
- net N$36: now also U$10.06_OUT1; no longer U$5.OUT1
- net N$38: now also D52.C
- net N$39: now also U$10.07_OUT2; no longer U$5.OUT2
- net N$4: now also D43.C
- net N$41: now also D53.C
- net N$42: now also U$10.08_OUT3; no longer U$5.OUT3
- net N$44: now also D54.C
- net N$45: now also U$10.09_OUT4; no longer U$5.OUT4
- net N$47: now also D55.C
- net N$48: now also U$10.10_OUT5; no longer U$5.OUT5
- net N$5: now also U$9.06_OUT1; no longer IC1.OUT1
- net N$50: now also D56.C
- net N$51: now also U$10.11_OUT6; no longer U$5.OUT6
- net N$53: now also D57.C
- net N$54: now also U$10.12_OUT7; no longer U$5.OUT7
- net N$56: now also D58.C
- net N$7: now also D44.C
- net N$8: now also U$9.07_OUT2; no longer IC1.OUT2
- net SDO1: now also U$9.02_SDI; no longer IC1.SDI
Other:
- moved on the sheet: D17, D9, R17, R18, R49, R50, R51, U$10, U$9

Commit message: diodak felkerultek
Connections:
- net +3V3: now also R23.2
- net +5V: no longer R23.2
Changed lines of the file:
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@@
 <part name="D20" library="microbuilder" deviceset="DIODE" device="SOD-323" value="1N4148"/>
 <part name="R23" library="rcl" deviceset="R-EU_" device="R0805" value="2k2"/>
-<part name="P+20" library="supply1" deviceset="+5V" device=""/>
 <part name="OK2" library="optocoupler" deviceset="TLP283-4" device="" value="TLP281-4"/>
 <part name="D21" library="microbuilder" deviceset="DIODE" device="SOD-323" value="1N4148"/>
@@
 <part name="D57" library="dp_devices" deviceset="DIODE" device="-SOD-123"/>
 <part name="D58" library="dp_devices" deviceset="DIODE" device="-SOD-123"/>
+<part name="+3V12" library="supply1" deviceset="+3V3" device=""/>
 </parts>
 <sheets>
@@
 <instance part="D20" gate="G$1" x="617.22" y="-139.7" rot="R90"/>
 <instance part="R23" gate="G$1" x="162.56" y="-218.44" rot="MR90"/>
-<instance part="P+20" gate="1" x="162.56" y="-208.28" rot="MR0"/>
 <instance part="OK2" gate="A" x="99.06" y="-228.6"/>
 <instance part="OK2" gate="B" x="99.06" y="-243.84"/>
@@
 <instance part="D57" gate="D" x="584.2" y="-114.3" rot="R90"/>
 <instance part="D58" gate="D" x="622.3" y="-114.3" rot="R90"/>
+<instance part="+3V12" gate="G$1" x="162.56" y="-208.28"/>
 </instances>
 <busses>
@@
 </segment>
 <segment>
-<pinref part="R23" gate="G$1" pin="2"/>
-<pinref part="P+20" gate="1" pin="+5V"/>
-<wire x1="162.56" y1="-210.82" x2="162.56" y2="-213.36" width="0.1524" layer="91"/>
-</segment>
-<segment>
 <pinref part="D21" gate="G$1" pin="C"/>
 <wire x1="83.82" y1="-226.06" x2="83.82" y2="-223.52" width="0.1524" layer="91"/>
@@
 <pinref part="+3V2" gate="G$1" pin="+3V3"/>
 </segment>
+<segment>
+<pinref part="R23" gate="G$1" pin="2"/>
+<pinref part="+3V12" gate="G$1" pin="+3V3"/>
+<wire x1="162.56" y1="-213.36" x2="162.56" y2="-210.82" width="0.1524" layer="91"/>
+</segment>
 </net>

Commit message: Streamnet finished
Connections:
- net CHECK: now also U$8.14_SDO; no longer U$8.13_!OE!
- net N$26: now also U$8.13_!OE!; no longer U$8.14_SDO
Changed lines of the file:
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@@
 2022 augusztus vége</text>
 <text x="655.32" y="-142.24" size="1.778" layer="91">BC807</text>
-<wire x1="134.62" y1="-317.5" x2="619.76" y2="-317.5" width="0.1524" layer="106"/>
 </plain>
 <instances>
@@
 <instance part="R51" gate="G$1" x="530.86" y="-335.28" rot="R180"/>
 <instance part="GND46" gate="1" x="320.04" y="-340.36"/>
-<instance part="GND47" gate="1" x="551.18" y="-340.36" smashed="yes">
-<attribute name="VALUE" x="548.64" y="-342.9" size="1.778" layer="96"/>
+<instance part="GND47" gate="1" x="558.8" y="-340.36" smashed="yes">
+<attribute name="VALUE" x="556.26" y="-342.9" size="1.778" layer="96"/>
 </instance>
 <instance part="GND48" gate="1" x="121.92" y="-340.36"/>
@@
 <segment>
 <pinref part="GND47" gate="1" pin="GND"/>
-<pinref part="U$8" gate="G$1" pin="14_SDO"/>
-<wire x1="551.18" y1="-337.82" x2="551.18" y2="-322.58" width="0.1524" layer="91"/>
-<wire x1="551.18" y1="-322.58" x2="546.1" y2="-322.58" width="0.1524" layer="91"/>
+<wire x1="558.8" y1="-337.82" x2="558.8" y2="-320.04" width="0.1524" layer="91"/>
+<pinref part="U$8" gate="G$1" pin="13_!OE!"/>
+<wire x1="546.1" y1="-320.04" x2="558.8" y2="-320.04" width="0.1524" layer="91"/>
 </segment>
 <segment>
@@
 <net name="CHECK" class="0">
 <segment>
-<wire x1="553.72" y1="-320.04" x2="553.72" y2="-360.68" width="0.1524" layer="91"/>
-<wire x1="553.72" y1="-360.68" x2="543.56" y2="-360.68" width="0.1524" layer="91"/>
+<wire x1="551.18" y1="-322.58" x2="551.18" y2="-360.68" width="0.1524" layer="91"/>
+<wire x1="551.18" y1="-360.68" x2="543.56" y2="-360.68" width="0.1524" layer="91"/>
 <label x="543.56" y="-360.68" size="1.27" layer="95" xref="yes"/>
-<pinref part="U$8" gate="G$1" pin="13_!OE!"/>
-<wire x1="546.1" y1="-320.04" x2="553.72" y2="-320.04" width="0.1524" layer="91"/>
+<pinref part="U$8" gate="G$1" pin="14_SDO"/>
+<wire x1="546.1" y1="-322.58" x2="551.18" y2="-322.58" width="0.1524" layer="91"/>
 </segment>
 <segment>
