File: stopper/Stopper_alap_V14_qfn.brd (EAGLE design)
At the start: 65.1 x 59.4 mm, 36 parts, among them CN1 PIN10_2, CN2 PIN10_2, CN3 PIN10_2, CN4 PIN03_1, CN5 PIN03_2'THT', CN6 PIN07_1, U1 MICROCHIP_PIC18F45K80-I-MLMIC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

Commit message: stopper elkeszult
Parts:
- added SJ1: (no value), jumper:SJ
- CANIC: value MCP2551 -> MCP2551/62
Connections:
- new net N$1: CANIC.5, SJ1.3
- net +5V: now also SJ1.2
Routing:
- net +5V: track 345.4 -> 355.0 mm, vias 2 -> 3
- net N$1: track 0.00 -> 2.54 mm
- net RB3: track 52.9 -> 50.7 mm
- net RB2: track 43.7 -> 42.3 mm
Other:
- board text added: "JP:62"
- board text added: "Stopper_alap V1.4"
- board text added: "V1.4"
- board text removed: "Stopper_alap V1.3"
- board text removed: "V1.3"
