File: stopper/Stopper_alap_V14_qfn.sch (EAGLE design)
At the start: 36 parts, among them CN1 PIN10_2, CN2 PIN10_2, CN3 PIN10_2, CN4 PIN03_1, CN5 PIN03_2'THT', CN6 PIN07_1, U1 MICROCHIP_PIC18F45K80-I-MLMIC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

Commit message: stopper elkeszult
Parts:
- added SJ1: (no value), jumper:SJ
- CANIC: value MCP2551 -> MCP2551/62
Connections:
- new net N$1: CANIC.VREF, SJ1.1
- net +5V: now also SJ1.2
Other:
- moved on the sheet: CN_CAN, CN_CANLEZAR, R4, R5
Changed lines of the file:
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@@
 <?xml version="1.0" encoding="utf-8"?>
 <!DOCTYPE eagle SYSTEM "eagle.dtd">
-<eagle version="7.5.0">
+<eagle version="6.5.0">
 <drawing>
 <settings>
@@
 <part name="GND16" library="supply1" deviceset="GND" device=""/>
 <part name="C28" library="Cf_RLCPX" deviceset="C" device="0805" value="100n"/>
-<part name="CANIC" library="Microchip_By_element14_Batch_1" deviceset="MCP2551-I/P" device="" value="MCP2551"/>
+<part name="CANIC" library="Microchip_By_element14_Batch_1" deviceset="MCP2551-I/P" device="" value="MCP2551/62"/>
 <part name="P+13" library="supply1" deviceset="+5V" device=""/>
 <part name="P+14" library="supply1" deviceset="+5V" device=""/>
@@
 <part name="U1" library="ML" deviceset="MICROCHIP_PIC18F45K80-I-ML" device="MICROCHIP_PIC18F45K80-I-ML_0_2"/>
 <part name="C5" library="Cf_RLCPX" deviceset="C" device="0805" value="100n"/>
+<part name="SJ1" library="jumper" deviceset="SJ" device=""/>
+<part name="P+4" library="supply1" deviceset="+5V" device=""/>
 </parts>
 <sheets>
@@
 <attribute name="VALUE" x="0" y="33.02" size="1.778" layer="96" rot="R90"/>
 </instance>
-<instance part="R5" gate="G$1" x="-20.32" y="10.16" smashed="yes" rot="R90">
-<attribute name="NAME" x="-24.13" y="11.049" size="1.778" layer="95"/>
-<attribute name="VALUE" x="-24.13" y="7.62" size="1.778" layer="96"/>
-</instance>
-<instance part="R4" gate="G$1" x="-20.32" y="15.24" smashed="yes" rot="R270">
-<attribute name="NAME" x="-24.13" y="16.129" size="1.778" layer="95"/>
-<attribute name="VALUE" x="-24.13" y="12.7" size="1.778" layer="96"/>
+<instance part="R5" gate="G$1" x="-35.56" y="10.16" smashed="yes" rot="R90">
+<attribute name="NAME" x="-39.37" y="11.049" size="1.778" layer="95"/>
+<attribute name="VALUE" x="-39.37" y="7.62" size="1.778" layer="96"/>
+</instance>
+<instance part="R4" gate="G$1" x="-35.56" y="15.24" smashed="yes" rot="R270">
+<attribute name="NAME" x="-39.37" y="16.129" size="1.778" layer="95"/>
+<attribute name="VALUE" x="-39.37" y="12.7" size="1.778" layer="96"/>
 </instance>
 <instance part="STAB1" gate="A1" x="-5.08" y="-15.24" smashed="yes">
@@
 <attribute name="VALUE" x="71.12" y="-15.24" size="1.778" layer="96" rot="R90"/>
 </instance>
-<instance part="GND19" gate="1" x="-58.42" y="10.16" smashed="yes" rot="MR0">
-<attribute name="VALUE" x="-55.88" y="7.62" size="1.778" layer="96" rot="MR0"/>
+<instance part="GND19" gate="1" x="-73.66" y="10.16" smashed="yes" rot="MR0">
+<attribute name="VALUE" x="-71.12" y="7.62" size="1.778" layer="96" rot="MR0"/>
 </instance>
 <instance part="Q1" gate="G$1" x="68.58" y="30.48" rot="R90"/>
@@
 <attribute name="VALUE" x="-27.94" y="-35.56" size="1.778" layer="96" rot="R90"/>
 </instance>
-<instance part="CN_CAN" gate="G$1" x="-50.8" y="5.08" rot="R180"/>
-<instance part="CN_CANLEZAR" gate="G$1" x="-33.02" y="12.7" rot="R180"/>
+<instance part="CN_CAN" gate="G$1" x="-66.04" y="5.08" rot="R180"/>
+<instance part="CN_CANLEZAR" gate="G$1" x="-48.26" y="12.7" rot="R180"/>
 <instance part="GND12" gate="1" x="279.4" y="12.7"/>
 <instance part="P+9" gate="1" x="266.7" y="20.32" smashed="yes">
@@
 <attribute name="NAME" x="80.899" y="-7.366" size="1.778" layer="95" rot="R180"/>
 <attribute name="VALUE" x="85.979" y="-1.016" size="1.778" layer="96" rot="R180"/>
+</instance>
+<instance part="SJ1" gate="1" x="-17.78" y="15.24" rot="R90"/>
+<instance part="P+4" gate="1" x="-17.78" y="25.4" smashed="yes">
+<attribute name="VALUE" x="-20.32" y="20.32" size="1.778" layer="96" rot="R90"/>
 </instance>
 </instances>
@@
 <segment>
 <pinref part="GND19" gate="1" pin="GND"/>
-<wire x1="-58.42" y1="12.7" x2="-43.18" y2="12.7" width="0.1524" layer="91"/>
-<wire x1="-43.18" y1="12.7" x2="-43.18" y2="7.62" width="0.1524" layer="91"/>
+<wire x1="-73.66" y1="12.7" x2="-58.42" y2="12.7" width="0.1524" layer="91"/>
+<wire x1="-58.42" y1="12.7" x2="-58.42" y2="7.62" width="0.1524" layer="91"/>
 <pinref part="CN_CAN" gate="G$1" pin="2"/>
 <pinref part="CN_CAN" gate="G$1" pin="1"/>
-<wire x1="-58.42" y1="7.62" x2="-43.18" y2="7.62" width="0.1524" layer="91"/>
+<wire x1="-73.66" y1="7.62" x2="-58.42" y2="7.62" width="0.1524" layer="91"/>
 </segment>
 <segment>
@@
 <label x="106.68" y="86.36" size="1.778" layer="95" rot="R180" xref="yes"/>
 </segment>
+<segment>
+<pinref part="SJ1" gate="1" pin="2"/>
+<pinref part="P+4" gate="1" pin="+5V"/>
+<wire x1="-17.78" y1="20.32" x2="-17.78" y2="22.86" width="0.1524" layer="91"/>
+</segment>
 </net>
 <net name="MCLR" class="0">
@@
 <net name="N$99" class="0">
 <segment>
-<wire x1="-12.7" y1="2.54" x2="-12.7" y2="12.7" width="0.1524" layer="91"/>
-<wire x1="-12.7" y1="12.7" x2="-25.4" y2="12.7" width="0.1524" layer="91"/>
+<wire x1="-27.94" y1="2.54" x2="-27.94" y2="12.7" width="0.1524" layer="91"/>
+<wire x1="-27.94" y1="12.7" x2="-40.64" y2="12.7" width="0.1524" layer="91"/>
 <pinref part="CANIC" gate="A" pin="CANH"/>
-<wire x1="-10.16" y1="2.54" x2="-12.7" y2="2.54" width="0.1524" layer="91"/>
-<junction x="-12.7" y="2.54"/>
-<wire x1="-12.7" y1="2.54" x2="-43.18" y2="2.54" width="0.1524" layer="91"/>
+<wire x1="-10.16" y1="2.54" x2="-27.94" y2="2.54" width="0.1524" layer="91"/>
+<junction x="-27.94" y="2.54"/>
+<wire x1="-27.94" y1="2.54" x2="-58.42" y2="2.54" width="0.1524" layer="91"/>
 <pinref part="CN_CAN" gate="G$1" pin="6"/>
 <pinref part="CN_CAN" gate="G$1" pin="5"/>
-<wire x1="-58.42" y1="2.54" x2="-43.18" y2="2.54" width="0.1524" layer="91"/>
+<wire x1="-73.66" y1="2.54" x2="-58.42" y2="2.54" width="0.1524" layer="91"/>
 <pinref part="CN_CANLEZAR" gate="G$1" pin="4"/>
 <pinref part="CN_CANLEZAR" gate="G$1" pin="3"/>
-<wire x1="-25.4" y1="12.7" x2="-40.64" y2="12.7" width="0.1524" layer="91"/>
-<junction x="-25.4" y="12.7"/>
+<wire x1="-40.64" y1="12.7" x2="-55.88" y2="12.7" width="0.1524" layer="91"/>
+<junction x="-40.64" y="12.7"/>
 </segment>
 </net>
 <net name="N$131" class="0">
 <segment>
-<wire x1="-15.24" y1="5.08" x2="-15.24" y2="10.16" width="0.1524" layer="91"/>
-<wire x1="-15.24" y1="10.16" x2="-15.24" y2="15.24" width="0.1524" layer="91"/>
+<wire x1="-30.48" y1="5.08" x2="-30.48" y2="10.16" width="0.1524" layer="91"/>
+<wire x1="-30.48" y1="10.16" x2="-30.48" y2="15.24" width="0.1524" layer="91"/>
 <pinref part="CANIC" gate="A" pin="CANL"/>
-<wire x1="-10.16" y1="5.08" x2="-15.24" y2="5.08" width="0.1524" layer="91"/>
+<wire x1="-10.16" y1="5.08" x2="-30.48" y2="5.08" width="0.1524" layer="91"/>
 <pinref part="R4" gate="G$1" pin="E"/>
 <pinref part="R5" gate="G$1" pin="A"/>
-<junction x="-15.24" y="10.16"/>
-<junction x="-15.24" y="5.08"/>
-<wire x1="-43.18" y1="5.08" x2="-15.24" y2="5.08" width="0.1524" layer="91"/>
+<junction x="-30.48" y="10.16"/>
+<junction x="-30.48" y="5.08"/>
+<wire x1="-58.42" y1="5.08" x2="-30.48" y2="5.08" width="0.1524" layer="91"/>
 <pinref part="CN_CAN" gate="G$1" pin="4"/>
 <pinref part="CN_CAN" gate="G$1" pin="3"/>
-<wire x1="-43.18" y1="5.08" x2="-58.42" y2="5.08" width="0.1524" layer="91"/>
+<wire x1="-58.42" y1="5.08" x2="-73.66" y2="5.08" width="0.1524" layer="91"/>
 </segment>
 </net>
@@
 <pinref part="CN_CANLEZAR" gate="G$1" pin="6"/>
 <pinref part="CN_CANLEZAR" gate="G$1" pin="5"/>
-<wire x1="-40.64" y1="10.16" x2="-25.4" y2="10.16" width="0.1524" layer="91"/>
-<junction x="-25.4" y="10.16"/>
+<wire x1="-55.88" y1="10.16" x2="-40.64" y2="10.16" width="0.1524" layer="91"/>
+<junction x="-40.64" y="10.16"/>
 </segment>
 </net>
@@
 <pinref part="CN_CANLEZAR" gate="G$1" pin="2"/>
 <pinref part="CN_CANLEZAR" gate="G$1" pin="1"/>
-<wire x1="-40.64" y1="15.24" x2="-25.4" y2="15.24" width="0.1524" layer="91"/>
-<junction x="-25.4" y="15.24"/>
+<wire x1="-55.88" y1="15.24" x2="-40.64" y2="15.24" width="0.1524" layer="91"/>
+<junction x="-40.64" y="15.24"/>
 </segment>
 </net>
@@
 </segment>
 </net>
+<net name="N$1" class="0">
+<segment>
+<pinref part="SJ1" gate="1" pin="1"/>
+<pinref part="CANIC" gate="A" pin="VREF"/>
+<wire x1="-17.78" y1="10.16" x2="-10.16" y2="10.16" width="0.1524" layer="91"/>
+</segment>
+</net>
